File: IMU Schematic/IMU Schematic.kicad_sch (KiCad schematic)
At the start: 1 part

Commit message: Correction to Schematic Drawing
Changed lines of the file:
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@@
 			)
 		)
-		(property "Value" "GY-9250 module (MPU-6500)"
+		(property "Value" "MPU-9250 module (MPU-6500)"
 			(at 191.77 74.93 0)
 			(show_name no)
